File: hardware/base/base.kicad_sch (KiCad schematic)
At the start: 70 parts, among them J1 SWD, J2 USB_B_Mini, J4 Serial Interface, J5 Debug, J5 OLED Display, J6 Conn_01x02_Pin, M1 Fan_ALT, Q1 Q_NMOS_GSD, Q2 Q_NMOS_GSD, Q3 Q_NMOS_GSD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

Commit message: Finish first hardware iteration (#3)
* Add Schottky rectifier symbol and footprint

* import components to PCB

* Fix relative paths

* Change transducer symbol

* Update PCB and Schema after symbol change

* Remove separate schematics

* did some layout and routing

CHANGELOG

* Changelog

* move humidifier to fan/SD_MODE control pin, small fixes

* Update README.md

* Add diode footprint

* finished placing components

* Update CHANGELOG.md

* Update CHANGELOG.md

* fix references

Co-authored-by: yuvve <yuvve@users.noreply.github.com>

* Add missing symbol

* Finish front layer traces

* Finish traces

Few warnings left

* add mounting holes

* Update CHANGELOG.md

---------

Co-authored-by: Simon Larsson <99037566+simlar-0@users.noreply.github.com>
Co-authored-by: filthytv <filthytv@ludd.ltu.se>
Parts:
- removed C21: 100 nF, Capacitor_SMD:C_0603_1608Metric, symbol Device:C
- removed D2: 1N4001, Diode_THT:D_DO-41_SOD81_P10.16mm_Horizontal, symbol Diode:1N4001
- removed D4, D5: D, symbol Device:D
- removed J6: Conn_01x02_Pin, symbol Connector:Conn_01x02_Pin
- removed L1: 300 uH, Inductor_SMD:L_0603_1608Metric, symbol Device:L
- removed Q4: MMBT2222A, Package_TO_SOT_SMD:SOT-23, symbol Transistor_BJT:MMBT2222A
- removed R11: 100 Ohm, Resistor_SMD:R_0603_1608Metric, symbol Device:R
- added D2, D3, D4: D_Schottky_1_3, Schottky Diode (ZLLS500TA):SOT91P240X110-3N, symbol SOT91P240X110-3N:D_Schottky_1_3
- added H1, H2, H3, H4: MountingHole, MountingHole:MountingHole_2.2mm_M2_ISO7380, symbol Mechanical:MountingHole
- added TP3, TP5, TP6: TestPoint, E7020E:TestPoint_THTPad_1.5x1.5mm_Drill0.8mm, symbol Connector:TestPoint
- added Y3: 1.70 MHz, Connector_PinHeader_2.54mm:PinHeader_1x02_P2.54mm_Vertical, symbol Device:Crystal
- B1: footprint HD-EMC1203-LW20-R:PUI_HD-EMC1203-LW20-R -> Connector_PinHeader_2.54mm:PinHeader_1x02_P2.54mm_Vertical
- BT1: footprint 796136-1:TE_796136-1 -> Battery Holder (796136-1):TE_796136-1
- C15: value 100 nF -> 10nF
- LS1: footprint (none) -> Connector_PinHeader_2.54mm:PinHeader_1x02_P2.54mm_Vertical
- R10: value 10kOhm -> 150 kOhm
- R11: renamed from RX1; value 664k -> 470 kOhm
- R5: value 100 Ohm -> 10k
- R7: value 100 Ohm -> 22 Ohm
- R9: value 132 kOhm -> 100 kOhm
Connections:
- net +3.3V: now also C16.1, J5.2 (Pin_2), D2.3 (K), D3.3 (K); no longer B1.P, C23.1
- net AMP_BCLK: now also TP5.1
- net AMP_DIN: now also TP4.1
- net AMP_LRCLK: now also TP6.1
- net DETECT_VSOURCE: now also U1.32 (AIN0/P0.02); no longer U1.22 (NFC1/P0.09)
- net GND: now also C15.2, Q3.2 (S), R5.2, U3.17 (PAD); no longer R10.2
- net ROT_ENC_S1: now also C15.1
- net VBUS: now also C23.1, R7.1, D4.3 (K), Y3.1
- net at C25.1, U4.3 (VO): now also D3.1 (A)
- net at C23.2: now also B1.2, Q3.3 (D), D4.1 (A); no longer B1.N
- net AMP_FAN_HUM: now reaches Q2.1 (G), R6.1, TP2.1, U1.23 (NFC2/P0.10)
- net AMP_FAN_HUM: now also R10.1; no longer R11.1
- net at BT1.1 (+): now also D2.1 (A)
- net at M1.1 (+), Q2.3 (D): now also Y3.2
- net LED: now reaches Q1.1 (G), R2.1
- net LED: now also TP1.1, U1.22 (NFC1/P0.09); no longer R7.2
- net HUMIDIFIER_MOSFET_GATE renamed HAPTIC
- net HAPTIC: now also TP3.1; no longer R10.1, R5.2, TP4.1
- removed net LED_HAPTIC: R7.1, TP1.1, U1.32 (AIN0/P0.02)
- new net: B1.1, R7.2
- new net: R10.2, R11.1
- no-connect marks 4 -> 3
Other:
- note removed: "3.3/5 = (132)/(68+132)"
- note removed: "BCLK, Serial clock, Freq = LRCLK * Bits_per_sample * Channels"
- note removed: "DIN = Serial data in"
- note removed: "Divide voltage to get 3.3V from 5V"
- note removed: "Exposed Pad. The exposed pad is not internally connected. Connect the exposed page to a solid ground plane for thermal dissipation."
- note removed: "LRCLK, Left-Right clock, Freq = Audio Sample Rate"
- note removed: "Operating Voltage Range: 2.5 ~ 3.5 V_{DC}"
- note removed: "SDMODE, To GPIO if we want to be able to turn OFF"
- note removed: "V_{out}= V_{in} * (R_{2})/(R_{1}+R_{2})"
- note removed: "http://www.learningaboutelectronics.com/Articles/Vibration-motor-circuit.php"
- moved on the sheet: B1, C10, C16, C19, C20, C23, C9, D1, LS1, M1, Q1, Q2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
